File: QCMAmplifier/QCMAmp.kicad_sch (KiCad schematic)
At the start: 55 parts, among them J1 Screw_Terminal_01x02, J2 Screw_Terminal_01x02, J3 Screw_Terminal_01x02, J4 Screw_Terminal_01x02, J5 Screw_Terminal_01x02, J6 Screw_Terminal_01x02, J7 Screw_Terminal_01x02, J8 Screw_Terminal_01x02, J9 Screw_Terminal_01x02, U1 PA119CE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

Commit message: changes in schematic
Parts:
- added H4: MountingHole, MountingHole:MountingHole_3.2mm_M3, symbol Mechanical:MountingHole
- C1, C12, C6, C9: value C -> 10uF
- C10, C3, C4, C7: value C -> 1nF
- C11, C2, C5, C8: value C -> 100nF
Connections:
- net OUT_LT: now also J3.2 (Pin_2), J4.1 (Pin_1), R15.1, R17.1; no longer R12.2, R14.2, R16.2, U2.7 (OUT)
- net OUT_PA: now also J5.2 (Pin_2), J6.1 (Pin_1), R3.1, R6.1, R9.1; no longer CC1.1, R1.2, R4.2, R7.2, RF1.1, RL1.1, U1.1 (OUT)
- removed net OUT: J3.2 (Pin_2), J4.1 (Pin_1), J5.2 (Pin_2), J6.1 (Pin_1), R15.1, R17.1, R3.1, R6.1, R9.1
- net VS1+ renamed +36V
- net VS1- renamed -36V
- net VS2+ renamed +15V
- net VS2- renamed -15V
- new net OUT_LT_R: R12.2, R14.2, R16.2, U2.7 (OUT)
- new net OUT_PA_R: CC1.1, R1.2, R4.2, R7.2, RF1.1, RL1.1, U1.1 (OUT)
Other:
- moved on the sheet: C12, C2, C3, C5, C6, C9, J5, J6, R14, R15, R16, R17

Commit message: changes made, gerbers added
Parts:
- added H5, H6, H7, H8: MountingHole, MountingHole:MountingHole_3.2mm_M3, symbol Mechanical:MountingHole
- J7: footprint TerminalBlock_4Ucon:TerminalBlock_4Ucon_1x02_P3.50mm_Vertical -> Connector_Coaxial:SMA_Amphenol_132134_Vertical
Connections:
- net GND: now also J7.2 (Pin_2); no longer J7.1 (Pin_1)
- net IN: now also J7.1 (Pin_1); no longer J7.2 (Pin_2)
